Commit message: planning usin ruckig

File: descriptions/robot_descriptions/excavator_bullet/excavatorplus.urdf (robot description, URDF)
Before this commit: robot excavatorplus, 5 links, 4 joints
Joints:
- joint joint1: limit lower=-3 upper=3 effort=100 velocity=1 -> lower=-2.5 upper=2.5 effort=100 velocity=1
